File: KiCad Files/LED Array PCB (LAP) v3.0/LAP-v3.0.kicad_pcb (KiCad board)
At the start: 2 copper layers, 114.3 x 89.2 mm, 61 parts, among them J1 DC37_Plug, U2 PCA9685PW

Commit message: Finalized PCBs
Other:
- board text added: "LED Array Controller"
- board text removed: "LED Array Controller v3.0"
Changed lines of the file:
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@@
     (effects (font (size 1 1) (thickness 0.15)) (justify left bottom))
   )
-  (gr_text "LED Array Controller v3.0" (at 186.944 189.992) (layer "F.SilkS")
+  (gr_text "LED Array Controller" (at 186.944 189.992) (layer "F.SilkS")
     (effects (font (size 1 1) (thickness 0.15)) (justify left bottom))
   )
