File: KiCad Files/LED Array PCB (LAP) v3.0/LAP-v3.0.kicad_sch (KiCad schematic)
At the start: 61 parts, among them J1 DC37_Plug, U2 PCA9685PW

Commit message: Finalized PCBs
Other:
- note added: "LED Array Controller"
- note removed: "LED Array Controller v3.0"
