File: KiCad Files/LED Array PCB (LAP) v4.0/LAP-v4.0.kicad_pcb (KiCad board)
At the start: 2 copper layers, 85.1 x 78.4 mm, 61 parts, among them J1 DC37_Plug_MountingHoles, U2 PCA9685PW

Commit message: Connected GND through-holes in LAP v4.0 to fix DRC error
Routing:
- net GND: track 56.8 -> 71.5 mm
Changed lines of the file:
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@@
   (via (at 86.995 83.185) (size 0.8) (drill 0.4) (layers "F.Cu" "B.Cu") (net 4))
   (via (at 114.935 47.625) (size 0.8) (drill 0.4) (layers "F.Cu" "B.Cu") (net 4))
+  (segment (start 138.83 76.2) (end 131.126191 83.903809) (width 0.25) (layer "B.Cu") (net 4))
+  (segment (start 131.126191 83.903809) (end 131.126191 87.68) (width 0.25) (layer "B.Cu") (net 4))
   (segment (start 132.845 108.885) (end 132.845 105.839009) (width 0.25) (layer "B.Cu") (net 5))
   (segment (start 154.07 58.42) (end 148.131149 64.358851) (width 0.25) (layer "B.Cu") (net 5))

Commit message: Finalized PCBs
Parts:
- moved ROE1 33.2 mm to (165.7, 102.3)
- moved C2_0 33.2 mm to (128.8, 83.2)
- moved C2_1 33.2 mm to (128.8, 92.7)
- moved R0 33.2 mm to (137.3, 71.3)
- moved R1 33.2 mm to (137.3, 75.4)
- moved R12 33.2 mm to (150.1, 71.3)
- moved R13 33.2 mm to (150.1, 75.4)
- moved R6 33.2 mm to (143.7, 71.3)
- moved R7 33.2 mm to (143.7, 75.4)
- moved U2 33.2 mm to (144.8, 61.3)
- moved C2_2 33.2 mm to (128.8, 102.3)
- moved C2_3 33.2 mm to (128.8, 111.8)
- moved A1 33.2 mm to (183.9, 93.3)
- moved C2_12 33.2 mm to (158.5, 83.2)
- moved C2_13 33.2 mm to (158.5, 92.7)
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Routing:
- net VCC: track 168.4 -> 174.0 mm
Other:
- board text added: "01/31/2025"
- board text added: "4"
- board text added: "L.Hanssler 20250131 v4.0 LED Array Controller"
- board text added: "LED Array Controller"
