File: KiCad Files/LED Array PCB (LAP) v4.0/LAP-v4.0.kicad_sch (KiCad schematic)
At the start: 61 parts, among them J1 DC37_Plug_MountingHoles, U2 PCA9685PW

Commit message: Finalized PCBs
Other:
- note added: "01/31/2025"
- note added: "4"
- note added: "LED Array Controller"
- note removed: "09/05/2024"
- note removed: "3"
- note removed: "LED Array Controller v3.0"
